Commit message: Update control.yaml in order to use Clearpath's diff_drive_controller. Add sensors to hibachi's urdf.

File: hibachi_description/xacro/hibachi.xacro (robot description, xacro)
@@ -73,3 +73,79 @@
         <origin xyz="${-wheel_distance/2} ${-wheel_separation/2} 0" rpy="0 0 0" />
     </xacro:hibachi_wheel>
+    <!-- LSM9DS1 IMU -->
+    <link name="imu_link"/>
+    <joint name="imu_joint" type="fixed">
+        <parent link="base_link" />
+        <child link="imu_link" />
+        <origin xyz="0 0 0.05" rpy="0 0 0" />
+    </joint>
+    <gazebo reference="imu_link"></gazebo>
+    <!-- MTI630 IMU -->
+    <link name="xsens_imu_link"/>
+    <joint name="xsens_imu_joint" type="fixed">
+        <parent link="base_link" />
+        <child link="xsens_imu_link" />
+        <origin xyz="0 0 0.1" rpy="0 0 0" />
+    </joint>
+    <!-- Phidget Spatial 3/3/3 IMU -->
+    <link name="phidgets_imu_link"/>
+    <joint name="phidgets_imu_joint" type="fixed">
+        <parent link="base_link" />
+        <child link="phidgets_imu_link" />
+        <origin xyz="0 0 0.1" rpy="0 0 0" />
+    </joint>
+    <!-- Ardusimple GPS Antenna -->
+    <link name="ardusimple_ant_link"/>
+    <joint name="ardusimple_ant_joint" type="fixed">
+        <parent link="base_link" />
+        <child link="ardusimple_ant_link" />
+        <origin xyz="0 0.05 0.28" rpy="0 0 0" />
+    </joint>
+    <!-- M8N GPS Antenna -->
+    <link name="m8n_ant_link"/>
+    <joint name="m8n_ant_joint" type="fixed">
+        <parent link="base_link" />
+        <child link="m8n_ant_link" />
+        <origin xyz="0 -0.05 0.28" rpy="0 0 0" />
+    </joint>
+    <!-- LiDAR -->
+    <link name="lidar_plate_link">
+        <visual>
+            <geometry>
+                <box size="0.2 0.2 0.005" />
+            </geometry>
+            <origin xyz="0 0 0" />
+        </visual>
+    </link>
+    <joint name="lidar_plate_joint" type="fixed">
+        <parent link="base_link" />
+        <child link="lidar_plate_link" />
+        <origin xyz="0 0 0.1" />
+    </joint>
+    <link name="rplidar_a1">
+        <collision>
+            <geometry>
+                <box size="96.8 70.3 55"/>
+            </geometry>
+            <origin xyz="0 0 0" />
+        </collision>
+        <visual>
+            <origin xyz="0 0 -0.05" rpy="0 0 0"/>
+            <geometry>
+                <mesh filename="package://hibachi_description/meshes/rplidar_a1.dae"  />
+            </geometry>
+        </visual>
+        <!-- Is this necessary? -->
+        <inertial>
+            <mass value="1e-5" />
+            <origin xyz="0 0 0" rpy="0 0 0"/>
+            <inertia ixx="0" ixy="0" ixz="0" iyy="0" iyz="0" izz="0" />
+        </inertial>
+    </link>
+    <joint name="rplidar_joint" type="fixed">
+        <parent link="lidar_plate_link"/>
+        <child link="rplidar_a1"/>
+        <axis xyz="0 1 0" />
+        <origin xyz="0 0 0.05" rpy="0 0 0"/>
+    </joint>
 </robot>
