Commit message: Rename simulated XSens output topic. Fix wheel color by updating material definition.

File: hibachi_description/urdf/hibachi_sim_sensors.urdf.xacro (robot description, xacro)
@@ -6,5 +6,5 @@
         <update_rate>20</update_rate>
         <visualize>true</visualize>
-        <topic>mti_630_8A1G6/imu/data</topic>
+        <topic>mti_630_8A1G6/imu/data_raw</topic>
         <gz_frame_id>xsens_imu_link</gz_frame_id>
         <!-- <enable_metrics>true</enable_metrics> -->
@@ -49,19 +49,4 @@
     </sensor>
 </gazebo>
-<!-- <gazebo>
-<plugin name="p3d_base_controller" filename="libgazebo_ros_p3d.so">
-    <alwaysOn>true</alwaysOn>
-    <updateRate>50.0</updateRate>
-    <robotNamespace>/</robotNamespace>
-    <bodyName>base_link</bodyName>
-    <body_name>base_link</body_name>
-    <frameId>base_link</frameId>
-    <topicName>ground_truth/state</topicName>
-    <gaussianNoise>0</gaussianNoise>
-    <frameName>world</frameName>
-    <xyzOffsets>0 0 0</xyzOffsets>
-    <rpyOffsets>0 0 0</rpyOffsets>
-</plugin>
-</gazebo> -->
 <gazebo reference="ardusimple_gps_link">
     <sensor name="ardusimple_navsat" type="navsat">

File: hibachi_description/urdf/wheel.urdf.xacro (robot description, xacro)
@@ -40,5 +40,15 @@
         </link>
         <gazebo reference="${link_name}">
-            <material>Gazebo/DarkGrey</material>
+            <visual>
+                <!-- Gazebo does not support Ogre material scripts
+                https://gazebosim.org/api/sim/8/migrationsdf.html#:~:text=Materials
+                https://github.com/gazebosim/gazebo-classic/blob/gazebo11/media/materials/scripts/gazebo.material
+                -->
+                <material>
+                    <ambient>0.175 0.175 0.175 1.0</ambient>
+                    <diffuse>0.175 0.175 0.175 1.0</diffuse>
+                    <specular>0.175 0.175 0.175 1.0</specular>
+                </material>
+            </visual>
             <!-- <selfCollide>false</selfCollide>
             <mu1 value="1.0"/>
