Commit message: Update robot description to match the metal frame. Add RPLidar S3 mesh.

File: hibachi_description/urdf/hibachi_core.urdf.xacro (robot description, xacro)
@@ -4,7 +4,7 @@
     <xacro:include filename="$(find hibachi_description)/urdf/wheel.urdf.xacro" />
 	<!--  Wheel distance between front and rear -->
-	<xacro:property name="wheel_distance" value="0.2" />
+	<xacro:property name="wheel_distance" value="0.25" />
 	<!-- Wheel distance between left and right side -->
-	<xacro:property name="wheel_separation" value="0.34" />
+	<xacro:property name="wheel_separation" value="0.475" />
 	<!-- Wheel properties -->
 	<xacro:property name="wheel_mass" value="0.150" />
@@ -12,13 +12,13 @@
 	<xacro:property name="wheel_width" value="0.06" />
 	<!-- Chassis size -->
-	<xacro:property name="chassis_x_size" value="0.40" />
-	<xacro:property name="chassis_y_size" value="0.25" />
+	<xacro:property name="chassis_x_size" value="0.45" />
+	<xacro:property name="chassis_y_size" value="0.38" />
 	<xacro:property name="chassis_z_size" value="0.05" />
 	<!-- https://docs.ros.org/en/humble/Tutorials/Intermediate/URDF/Adding-Physical-and-Collision-Properties-to-a-URDF-Model.html -->
     <link name="base_link">
 		<visual>
-    		<origin xyz="0 0 0.0278" rpy="${(pi/2)} 0 ${-(pi/2)}"/>
+    		<origin xyz="0 0 0" rpy="0 0 0" />
 			<geometry>
-				<mesh filename="file://$(find hibachi_description)/meshes/hibachi_chassis.stl" scale="0.001 0.001 0.001" />
+				<box size="${chassis_x_size} ${chassis_y_size} ${chassis_z_size}"/>
 			</geometry>
 			<material name="Red">
@@ -30,4 +30,19 @@
 			<geometry>
 				<box size="${chassis_x_size} ${chassis_y_size} ${chassis_z_size}"/>
+			</geometry>
+		</collision>
+		<visual>
+    		<origin xyz="${chassis_x_size/2 + 0.045} 0 ${chassis_z_size/2 + 0.06}" rpy="0 0 0" />
+			<geometry>
+				<box size="0.09 0.17 0.12"/>
+			</geometry>
+			<material name="Green">
+				<color rgba="${0/255} ${255/255} ${0/255} 1.0"/>
+			</material>
+		</visual>
+		<collision>
+			<origin xyz="${chassis_x_size/2 + 0.045} 0 ${chassis_z_size/2 + 0.06}" rpy="0 0 0" />
+			<geometry>
+				<box size="0.09 0.17 0.12"/>
 			</geometry>
 		</collision>
@@ -76,16 +91,17 @@
 		<origin xyz="0 0 0.05" rpy="0 0 0" />
 	</joint>
-	<!-- RPLidar A1 -->
-	<link name="rplidar_a1_link">
+	<!-- RPLidar S3 -->
+	<link name="rplidar_s3_link">
 		<xacro:dummy_inertial />
 		<collision>
-			<origin xyz="0 0 0.0275" rpy="0 0 0"/>
+			<origin xyz="0 0 0" rpy="0 0 0"/>
 			<geometry>
-				<box size="0.0968 0.0703 0.0550"/>
+				<box size="0.06 0.056 0.042"/>
 			</geometry>
 		</collision>
 		<visual>
+			<origin xyz="0 0 0" rpy="${pi/2} 0 ${-pi/2}"/>
 			<geometry>
-				<mesh filename="file://$(find hibachi_description)/meshes/rplidar_a1.dae"  />
+				<mesh filename="file://$(find hibachi_description)/meshes/rplidar_s3.stl"  scale="0.001 0.001 0.001"/>
 			</geometry>
 		</visual>
@@ -93,6 +109,6 @@
 	<joint name="rplidar_joint" type="fixed">
 		<parent link="base_link"/>
-		<child link="rplidar_a1_link"/>
-		<origin xyz="0 0 0.12" rpy="0 0 0"/>
+		<child link="rplidar_s3_link"/>
+		<origin xyz="0.1 0 ${chassis_z_size/2 + 0.16}" rpy="0 0 0"/>
 	</joint>
 	<link name="ardusimple_gps_link">

Commit message: Update URDF to the metal frame.

File: hibachi_description/urdf/hibachi_core.urdf.xacro (robot description, xacro)
@@ -110,5 +110,5 @@
 		<parent link="base_link"/>
 		<child link="rplidar_s3_link"/>
-		<origin xyz="0.1 0 ${chassis_z_size/2 + 0.16}" rpy="0 0 0"/>
+		<origin xyz="0.0 0.0 ${chassis_z_size/2 + 0.16}" rpy="0 0 ${pi}"/>
 	</joint>
 	<link name="ardusimple_gps_link">
